File: peoplecounter-pcb/peoplecounter-pcb.kicad_pcb (KiCad board)
At the start: 2 copper layers, 120 x 50 mm, 29 parts, among them J2 USB_C_Receptacle_USB2.0_16P, SW1 SW_DIP_x01, U1 VL53L0CXV0DH1, U2 VL53L0CXV0DH1, U3 AP2127K-2.8, U4 ESP32-S3-WROOM-1, U5 AMS1117-3.3

Commit message: update
Parts:
- removed REF** (x4): MountingHole_4mm_Pad_TopBottom, MountingHole:MountingHole_4mm_Pad_TopBottom
- removed U4: ESP32-S3-WROOM-1, PCM_Espressif:ESP32-S3-WROOM-1
- added U6: ESP32-C3-WROOM-02, PCM_Espressif:ESP32-C3-WROOM-02, F.Cu at (160.2, 94.9)
