File: peoplecounter-pcb/peoplecounter-pcb.kicad_sch (KiCad schematic)
At the start: 25 parts, among them J2 USB_C_Receptacle_USB2.0_16P, SW1 SW_DIP_x01, U1 VL53L0CXV0DH1, U2 VL53L0CXV0DH1, U3 AP2127K-2.8, U4 ESP32-S3-WROOM-1, U5 AMS1117-3.3

Commit message: update
Parts:
- removed D1: LED_RBGA, LED_SMD:LED_Kingbright_AAA3528ESGCT, symbol Device:LED_RBGA
- removed U4: ESP32-S3-WROOM-1, PCM_Espressif:ESP32-S3-WROOM-1, symbol PCM_Espressif:ESP32-S3-WROOM-1
- added U6: ESP32-C3-WROOM-02, PCM_Espressif:ESP32-C3-WROOM-02, symbol PCM_Espressif:ESP32-C3-WROOM-02
Connections:
- new net: U6.19 (GND), U6.9 (GND)
